File: HW2/PCB/pcb_schematic.sch (EAGLE design)
At the start: 20 parts, among them J1 USB-MB-H

Commit message: PCB is closer.
Parts:
- added U$8, U$9: SWITCH, pcb_library:SWITCH
Connections:
- net B4/USER: now also U$8.1.IN
- net GND: now also U$8.2.IN, U$9.2.IN
- net MCLR: now also U$9.1.IN
Changed lines of the file:
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@@
 <part name="R3" library="pcb_library" deviceset="R-US_" device="0204/7" value="10K"/>
 <part name="R4" library="pcb_library" deviceset="R-US_" device="0204/7" value="10K"/>
+<part name="U$8" library="pcb_library" deviceset="SWITCH" device=""/>
+<part name="U$9" library="pcb_library" deviceset="SWITCH" device=""/>
 </parts>
 <sheets>
@@
 <instance part="R3" gate="G$1" x="109.22" y="76.2" rot="R90"/>
 <instance part="R4" gate="G$1" x="109.22" y="43.18" rot="R90"/>
+<instance part="U$8" gate="G$1" x="129.54" y="68.58"/>
+<instance part="U$9" gate="G$1" x="129.54" y="35.56"/>
 </instances>
 <busses>
@@
 <segment>
 <pinref part="GND8" gate="1" pin="GND"/>
-<wire x1="119.38" y1="63.5" x2="109.22" y2="63.5" width="0.1524" layer="91"/>
+<wire x1="124.46" y1="63.5" x2="109.22" y2="63.5" width="0.1524" layer="91"/>
+<pinref part="U$8" gate="G$1" pin="2.IN"/>
 </segment>
 <segment>
 <pinref part="GND9" gate="1" pin="GND"/>
-<wire x1="116.84" y1="30.48" x2="109.22" y2="30.48" width="0.1524" layer="91"/>
+<pinref part="U$9" gate="G$1" pin="2.IN"/>
+<wire x1="124.46" y1="30.48" x2="109.22" y2="30.48" width="0.1524" layer="91"/>
 </segment>
 <segment>
@@
 <wire x1="96.52" y1="38.1" x2="109.22" y2="38.1" width="0.1524" layer="91"/>
 <label x="99.06" y="38.1" size="1.778" layer="95"/>
+<pinref part="U$9" gate="G$1" pin="1.IN"/>
+<wire x1="109.22" y1="38.1" x2="124.46" y2="38.1" width="0.1524" layer="91"/>
+<wire x1="124.46" y1="38.1" x2="124.46" y2="40.64" width="0.1524" layer="91"/>
+<junction x="109.22" y="38.1"/>
 </segment>
 </net>
@@
 <wire x1="96.52" y1="71.12" x2="109.22" y2="71.12" width="0.1524" layer="91"/>
 <label x="99.06" y="71.12" size="1.778" layer="95"/>
-</segment>
-</net>
+<pinref part="U$8" gate="G$1" pin="1.IN"/>
+<wire x1="109.22" y1="71.12" x2="124.46" y2="71.12" width="0.1524" layer="91"/>
+<wire x1="124.46" y1="71.12" x2="124.46" y2="73.66" width="0.1524" layer="91"/>
+<junction x="109.22" y="71.12"/>
+</segment>
+</net>
